File: pcb_layout/lora_sensor.sch (KiCad schematic (older format))
At the start: 71 parts, among them P4 USB_A, Q1 NXP BSS84, Q2 NXP 2N7002,215, Q3 NXP BSS84, U1 MCP73831/2, U2 PIC18F2XJ50, U3 TPS736, U4 BH1603FVC, U6 MCP9700T-E, U7 RN2483, Y1 16Mhz

Commit message: Updates Schematic
Parts:
- added R25, R26: 0, symbol R
- BATTERY1: footprint (none) -> Socket_Strips:Socket_Strip_Straight_1x02_Pitch2.54mm
- C1, C10, C11, C12, C13, C14, C15, C2, C3, C4, C5, C6, C7, C8, C9: footprint (none) -> Capacitors_SMD:C_0805
- C16, C17: renamed from C?; footprint (none) -> Capacitors_SMD:C_0805
- LED0, LED1, LED2, LED3, RF_LED_0, RF_LED_1: footprint (none) -> LEDs:LED_0805
- R1, R10, R12, R13, R14, R15, R16, R17, R18, R19, R2, R20, R21, R22, R23, R24, R3, R4, R5, R6, R7, R8, R9: footprint (none) -> Resistors_SMD:R_0805
Connections:
- net labels removed: PGM
- wire segments 243 -> 249
- no-connect marks 26 -> 27
Other:
- moved on the sheet: Battery_Current1, Charge_Current1

Commit message: Improved schematic, updated component-module mappings
Parts:
- removed BATTERY1: CONN_01X02, Socket_Strips:Socket_Strip_Straight_1x02_Pitch2.54mm, symbol CONN_01X02
- removed BUTTON_0, BUTTON_1: SwitchTactile, symbol SwitchTactile
- removed Battery_Current1, Charge_Current1, MCU_Current1, RF_Current1, RF_High1, RF_Low1: CONN_01X02, symbol CONN_01X02
- removed C1: 10uF, Capacitors_SMD:C_0805, symbol C
- removed C10, C15, C16: 1uF, Capacitors_SMD:C_0805, symbol C
- removed C11, C12, C13, C14, C6, C7, C8, C9: 100nF, Capacitors_SMD:C_0805, symbol C
- removed C17: 4.7u, Capacitors_SMD:C_0805, symbol C
- removed C2, C5: 10pF, Capacitors_SMD:C_0805, symbol C
- removed C3: 10nF, Capacitors_SMD:C_0805, symbol C
- removed C4: 4.7uF, Capacitors_SMD:C_0805, symbol C
- removed D1: D_Zener, symbol D_Zener
- removed D2: LED, symbol LED
- removed LED0, LED1, LED2, LED3, RF_LED_0, RF_LED_1: LED, LEDs:LED_0805, symbol LED
- removed P4: USB_A, symbol USB_A
- removed PICKIT3: CONN_01X06, symbol CONN_01X06
- removed Q1, Q3: NXP BSS84, symbol Q_PMOS_GSD
- removed Q2: NXP 2N7002,215, symbol Q_NMOS_DSG
- removed R1: 4k7, Resistors_SMD:R_0805, symbol R
- removed R10, R7: 47k, Resistors_SMD:R_0805, symbol R
- removed R11: R_Variable, symbol R_Variable
- removed R12, R13, R16, R17, R19, R20: 0, Resistors_SMD:R_0805, symbol R
- removed R14, R15, R18, R21, R22, R9: R, Resistors_SMD:R_0805, symbol R
- removed R2: 330, Resistors_SMD:R_0805, symbol R
- removed R23, R24, R3, R4, R8: 10k, Resistors_SMD:R_0805, symbol R
- removed R25, R26: 0, symbol R
- removed R5: 470, Resistors_SMD:R_0805, symbol R
- removed R6: 2k, Resistors_SMD:R_0805, symbol R
- removed U1: MCP73831/2, symbol MCP73831/2
- removed U2: PIC18F2XJ50, symbol PIC18F2XJ50
- removed U3: TPS736, symbol TPS736
- removed U4: BH1603FVC, symbol BH1603FVC
- removed U6: MCP9700T-E, symbol MCP9700T-E
- removed U7: RN2483, symbol RN2483
- removed UART2_CONN1: CONN_01X03, symbol CONN_01X03
- removed Y1: 16Mhz, symbol Crystal_GND23
Connections:
- net labels removed: +3.3V, AN0_batt, AN1_LDR, AN2_Ambient, AN3_Temp, BUTTON_0, BUTTON_1, Battery_input, GND, LED0, LED1, LED2, LED3, MCU_POW, OSC1, OSC2, PGC, PGD, RF_LED_0, RF_LED_1, RF_POW, RF_Reset, RF_Setting_0, RF_Setting_1, Sensors_Enable, UART_2_RX, UART_2_TX, UART_RX, UART_TX, USB_D+, USB_D-, VB_Control, VDD_Target, VPP/~MCLR, VSS, VUSB, V_Battery, V_CAP
- wire segments 249 -> 42
- no-connect marks 27 -> 0

Commit message: Added PCB LAyout
Parts:
- added J1, J2, J3: CONN_01X01, Mounting_Holes:MountingHole_3.2mm_M3_Pad, symbol CONN_01X01
Connections:
- no-connect marks 0 -> 3
Changed lines of the file:
@@
 LIBS:mcp9700t-e
 LIBS:rn2483
+LIBS:fa_238
 LIBS:lora_sensor-cache
-EELAYER 25 0
+EELAYER 26 0
 EELAYER END
 $Descr A4 11693 8268
@@
 F1 "power_section.sch" 60
 F2 "V_Battery" I R 3200 1550 60
-F3 "Gnd" I R 3200 2150 60
-F4 "RF_Power" I R 3200 1900 60
-F5 "MCU_Power" I R 3200 2000 60
-F6 "3.3V" I R 3200 1750 60
-F7 "V_USB" I R 3200 1650 60
+F3 "RF_Power" I R 3200 1900 60
+F4 "MCU_Power" I R 3200 2000 60
+F5 "3.3V" I R 3200 1750 60
+F6 "V_USB" I R 3200 1650 60
+F7 "GND" I R 3200 2150 60
 $EndSheet
 $Sheet
@@
 Wire Wire Line
 	7450 5500 6550 5500
+$Comp
+L CONN_01X01 J1
+U 1 1 589F7D41
+P 1650 6250
+F 0 "J1" H 1728 6291 50  0000 L CNN
+F 1 "CONN_01X01" H 1728 6200 50  0000 L CNN
+F 2 "Mounting_Holes:MountingHole_3.2mm_M3_Pad" H 100 1200 50  0001 C CNN
+F 3 "" H 100 1200 50  0001 C CNN
+	1    1650 6250
+	1    0    0    -1
+$EndComp
+$Comp
+L CONN_01X01 J2
+U 1 1 589F8006
+P 1650 6450
+F 0 "J2" H 1728 6491 50  0000 L CNN
+F 1 "CONN_01X01" H 1728 6400 50  0000 L CNN
+F 2 "Mounting_Holes:MountingHole_3.2mm_M3_Pad" H 100 1400 50  0001 C CNN
+F 3 "" H 100 1400 50  0001 C CNN
+	1    1650 6450
+	1    0    0    -1
+$EndComp
+$Comp
+L CONN_01X01 J3
+U 1 1 589F80EC
+P 1650 6650
+F 0 "J3" H 1728 6691 50  0000 L CNN
+F 1 "CONN_01X01" H 1728 6600 50  0000 L CNN
+F 2 "Mounting_Holes:MountingHole_3.2mm_M3_Pad" H 100 1600 50  0001 C CNN
+F 3 "" H 100 1600 50  0001 C CNN
+	1    1650 6650
+	1    0    0    -1
+$EndComp
+NoConn ~ 1450 6250
+NoConn ~ 1450 6450
+NoConn ~ 1450 6650
 $EndSCHEMATC
