File: pcb_layout/microcontroller.sch (KiCad schematic (older format))
At the start: 26 parts, among them P1 USB_A, U4 PIC18F2XJ50, Y1 16Mhz

Commit message: More modules, initial pcb layout
Parts:
- BUTTON_1, BUTTON_2: footprint (none) -> Buttons_Switches_SMD:SW_SPST_REED_CT05-XXXX-G1
- C10, C11: value 10pF -> 22pF
- C13: footprint Capacitors_SMD:C_0805 -> Capacitors_SMD:C_1206
- R18, R19, R20, R21: value R -> 330
- Y1: footprint (none) -> Crystals:Crystal_SMD_EuroQuartz_MQ-4pin_7.0x5.0mm_HandSoldering
- renumbered LED1 to LED0, LED2 to LED1, LED3 to LED2, LED4 to LED3
Other:
- note added: "The LED resistor values can be adjusted \nbased on the LEDs that are used."
Changed lines of the file:
@@
 $EndComp
 $Comp
-L GND #PWR26
+L GND #PWR022
 U 1 1 589BC9D0
 P 3450 3850
-F 0 "#PWR26" H 3450 3600 50  0001 C CNN
+F 0 "#PWR022" H 3450 3600 50  0001 C CNN
 F 1 "GND" H 3450 3700 50  0000 C CNN
 F 2 "" H 3450 3850 50  0000 C CNN
@@
 $EndComp
 $Comp
-L GND #PWR27
+L GND #PWR023
 U 1 1 589BC9DC
 P 3950 4200
-F 0 "#PWR27" H 3950 3950 50  0001 C CNN
+F 0 "#PWR023" H 3950 3950 50  0001 C CNN
 F 1 "GND" H 3950 4050 50  0000 C CNN
 F 2 "" H 3950 4200 50  0000 C CNN
@@
 $EndComp
 $Comp
-L GND #PWR33
+L GND #PWR024
 U 1 1 589BC9E2
 P 8850 4350
-F 0 "#PWR33" H 8850 4100 50  0001 C CNN
+F 0 "#PWR024" H 8850 4100 50  0001 C CNN
 F 1 "GND" H 8850 4200 50  0000 C CNN
 F 2 "" H 8850 4350 50  0000 C CNN
@@
 MCU_POW
 $Comp
-L GND #PWR31
+L GND #PWR025
 U 1 1 589BC9F7
 P 6100 1800
-F 0 "#PWR31" H 6100 1550 50  0001 C CNN
+F 0 "#PWR025" H 6100 1550 50  0001 C CNN
 F 1 "GND" H 6100 1650 50  0000 C CNN
 F 2 "" H 6100 1800 50  0000 C CNN
@@
 USB_D-
 $Comp
-L GND #PWR25
+L GND #PWR026
 U 1 1 589BCA03
 P 2450 7000
-F 0 "#PWR25" H 2450 6750 50  0001 C CNN
+F 0 "#PWR026" H 2450 6750 50  0001 C CNN
 F 1 "GND" H 2450 6850 50  0000 C CNN
 F 2 "" H 2450 7000 50  0000 C CNN
@@
 F 0 "Y1" H 1675 3750 50  0000 L CNN
 F 1 "16Mhz" H 1675 3675 50  0000 L CNN
-F 2 "" H 1550 3550 50  0001 C CNN
+F 2 "Crystals:Crystal_SMD_EuroQuartz_MQ-4pin_7.0x5.0mm_HandSoldering" H 1550 3550 50  0001 C CNN
 F 3 "" H 1550 3550 50  0000 C CNN
 	1    1550 3550
@@
 $EndComp
 $Comp
-L GND #PWR22
+L GND #PWR027
 U 1 1 589BCA14
 P 1550 4100
-F 0 "#PWR22" H 1550 3850 50  0001 C CNN
+F 0 "#PWR027" H 1550 3850 50  0001 C CNN
 F 1 "GND" H 1550 3950 50  0000 C CNN
 F 2 "" H 1550 4100 50  0000 C CNN
@@
 P 1800 3800
 F 0 "C11" H 1825 3900 50  0000 L CNN
-F 1 "10pF" H 1825 3700 50  0000 L CNN
+F 1 "22pF" H 1825 3700 50  0000 L CNN
 F 2 "Capacitors_SMD:C_0805" H 1838 3650 50  0001 C CNN
 F 3 "" H 1800 3800 50  0000 C CNN
@@
 P 1300 3800
 F 0 "C10" H 1325 3900 50  0000 L CNN
-F 1 "10pF" H 1325 3700 50  0000 L CNN
+F 1 "22pF" H 1325 3700 50  0000 L CNN
 F 2 "Capacitors_SMD:C_0805" H 1338 3650 50  0001 C CNN
 F 3 "" H 1300 3800 50  0000 C CNN
@@
 $EndComp
 $Comp
-L GND #PWR24
+L GND #PWR028
 U 1 1 589BCA28
 P 1750 3150
-F 0 "#PWR24" H 1750 2900 50  0001 C CNN
+F 0 "#PWR028" H 1750 2900 50  0001 C CNN
 F 1 "GND" H 1750 3000 50  0000 C CNN
 F 2 "" H 1750 3150 50  0000 C CNN
@@
 $EndComp
 $Comp
-L GND #PWR28
+L GND #PWR029
 U 1 1 589BCA2E
 P 4300 6600
-F 0 "#PWR28" H 4300 6350 50  0001 C CNN
+F 0 "#PWR029" H 4300 6350 50  0001 C CNN
 F 1 "GND" H 4300 6450 50  0000 C CNN
 F 2 "" H 4300 6600 50  0000 C CNN
@@
 F 0 "C13" H 4325 6500 50  0000 L CNN
 F 1 "10uF" H 4325 6300 50  0000 L CNN
-F 2 "Capacitors_SMD:C_0805" H 4338 6250 50  0001 C CNN
+F 2 "Capacitors_SMD:C_1206" H 4338 6250 50  0001 C CNN
 F 3 "" H 4300 6400 50  0000 C CNN
 	1    4300 6400
@@
 $EndComp
 $Comp
-L GND #PWR32
+L GND #PWR030
 U 1 1 589BCA42
 P 7600 1700
-F 0 "#PWR32" H 7600 1450 50  0001 C CNN
+F 0 "#PWR030" H 7600 1450 50  0001 C CNN
 F 1 "GND" H 7600 1550 50  0000 C CNN
 F 2 "" H 7600 1700 50  0000 C CNN
@@
 UART_2_TX
 $Comp
-L LED LED4
+L LED LED3
 U 1 1 589BCA4A
 P 10850 4500
-F 0 "LED4" H 10850 4600 50  0000 C CNN
+F 0 "LED3" H 10850 4600 50  0000 C CNN
 F 1 "LED" H 10850 4400 50  0000 C CNN
 F 2 "LEDs:LED_0805" H 10850 4500 50  0001 C CNN
@@
 $EndComp
 $Comp
-L LED LED3
+L LED LED2
 U 1 1 589BCA51
 P 10550 4500
-F 0 "LED3" H 10550 4600 50  0000 C CNN
+F 0 "LED2" H 10550 4600 50  0000 C CNN
 F 1 "LED" H 10550 4400 50  0000 C CNN
 F 2 "LEDs:LED_0805" H 10550 4500 50  0001 C CNN
@@
 P 10850 4100
 F 0 "R21" V 10930 4100 50  0000 C CNN
-F 1 "R" V 10850 4100 50  0000 C CNN
+F 1 "330" V 10850 4100 50  0000 C CNN
 F 2 "Resistors_SMD:R_0805" V 10780 4100 50  0001 C CNN
 F 3 "" H 10850 4100 50  0000 C CNN
@@
 P 10550 4100
 F 0 "R20" V 10630 4100 50  0000 C CNN
-F 1 "R" V 10550 4100 50  0000 C CNN
+F 1 "330" V 10550 4100 50  0000 C CNN
 F 2 "Resistors_SMD:R_0805" V 10480 4100 50  0001 C CNN
 F 3 "" H 10550 4100 50  0000 C CNN
@@
 P 10250 4100
 F 0 "R19" V 10330 4100 50  0000 C CNN
-F 1 "R" V 10250 4100 50  0000 C CNN
+F 1 "330" V 10250 4100 50  0000 C CNN
 F 2 "Resistors_SMD:R_0805" V 10180 4100 50  0001 C CNN
 F 3 "" H 10250 4100 50  0000 C CNN
@@
 $EndComp
 $Comp
-L LED LED2
+L LED LED1
 U 1 1 589BCA6D
 P 10250 4500
-F 0 "LED2" H 10250 4600 50  0000 C CNN
+F 0 "LED1" H 10250 4600 50  0000 C CNN
 F 1 "LED" H 10250 4400 50  0000 C CNN
 F 2 "LEDs:LED_0805" H 10250 4500 50  0001 C CNN
@@
 $EndComp
 $Comp
-L LED LED1
+L LED LED0
 U 1 1 589BCA74
 P 9950 4500
-F 0 "LED1" H 9950 4600 50  0000 C CNN
+F 0 "LED0" H 9950 4600 50  0000 C CNN
 F 1 "LED" H 9950 4400 50  0000 C CNN
 F 2 "LEDs:LED_0805" H 9950 4500 50  0001 C CNN
@@
 P 9950 4100
 F 0 "R18" V 10030 4100 50  0000 C CNN
-F 1 "R" V 9950 4100 50  0000 C CNN
+F 1 "330" V 9950 4100 50  0000 C CNN
 F 2 "Resistors_SMD:R_0805" V 9880 4100 50  0001 C CNN
 F 3 "" H 9950 4100 50  0000 C CNN
@@
 $EndComp
 $Comp
-L GND #PWR34
+L GND #PWR031
 U 1 1 589BCA82
 P 10850 4750
-F 0 "#PWR34" H 10850 4500 50  0001 C CNN
+F 0 "#PWR031" H 10850 4500 50  0001 C CNN
 F 1 "GND" H 10850 4600 50  0000 C CNN
 F 2 "" H 10850 4750 50  0000 C CNN
@@
 V_CAP
 $Comp
-L GND #PWR30
+L GND #PWR032
 U 1 1 589BCA8B
 P 4850 1600
-F 0 "#PWR30" H 4850 1350 50  0001 C CNN
+F 0 "#PWR032" H 4850 1350 50  0001 C CNN
 F 1 "GND" H 4850 1450 50  0000 C CNN
 F 2 "" H 4850 1600 50  0000 C CNN
@@
 F 0 "BUTTON_2" H 10450 2800 60  0000 C CNN
 F 1 "SwitchTactile" H 10450 3050 60  0000 C CNN
-F 2 "" H 10450 2900 60  0001 C CNN
+F 2 "Buttons_Switches_SMD:SW_SPST_REED_CT05-XXXX-G1" H 10450 2900 60  0001 C CNN
 F 3 "" H 10450 2900 60  0001 C CNN
 	1    10450 2900
@@
 $EndComp
 $Comp
-L GND #PWR36
+L GND #PWR033
 U 1 1 589BCAA4
 P 10900 3000
-F 0 "#PWR36" H 10900 2750 50  0001 C CNN
+F 0 "#PWR033" H 10900 2750 50  0001 C CNN
 F 1 "GND" H 10900 2850 50  0000 C CNN
 F 2 "" H 10900 3000 50  0000 C CNN
@@
 F 0 "BUTTON_1" H 10450 2050 60  0000 C CNN
 F 1 "SwitchTactile" H 10450 2300 60  0000 C CNN
-F 2 "" H 10450 2150 60  0001 C CNN
+F 2 "Buttons_Switches_SMD:SW_SPST_REED_CT05-XXXX-G1" H 10450 2150 60  0001 C CNN
 F 3 "" H 10450 2150 60  0001 C CNN
 	1    10450 2150
@@
 $EndComp
 $Comp
-L GND #PWR35
+L GND #PWR034
 U 1 1 589BCABA
 P 10900 2250
-F 0 "#PWR35" H 10900 2000 50  0001 C CNN
+F 0 "#PWR034" H 10900 2000 50  0001 C CNN
 F 1 "GND" H 10900 2100 50  0000 C CNN
 F 2 "" H 10900 2250 50  0000 C CNN
@@
 $EndComp
 $Comp
-L GND #PWR29
+L GND #PWR035
 U 1 1 589BCAD8
 P 4700 5150
-F 0 "#PWR29" H 4700 4900 50  0001 C CNN
+F 0 "#PWR035" H 4700 4900 50  0001 C CNN
 F 1 "GND" H 4700 5000 50  0000 C CNN
 F 2 "" H 4700 5150 50  0000 C CNN
@@
 V_USB
 $Comp
-L GND #PWR23
+L GND #PWR036
 U 1 1 589BCB64
 P 1600 1250
-F 0 "#PWR23" H 1600 1000 50  0001 C CNN
+F 0 "#PWR036" H 1600 1000 50  0001 C CNN
 F 1 "GND" H 1600 1100 50  0000 C CNN
 F 2 "" H 1600 1250 50  0000 C CNN
@@
 Wire Wire Line
 	3450 2900 4000 2900
+Text Notes 9300 5150 0    60   ~ 0
+The LED resistor values can be adjusted \nbased on the LEDs that are used.
 $EndSCHEMATC

Commit message: Added PCB LAyout
Parts:
- removed Y1: 16Mhz, Crystals:Crystal_SMD_EuroQuartz_MQ-4pin_7.0x5.0mm_HandSoldering, symbol Crystal_GND23
- added Y1: FA_238, libraries:Crystal_FA-238, symbol FA_238
- LED0, LED1, LED2, LED3: symbol LED -> LED-RESCUE-lora_sensor
- P1: symbol USB_A -> USB_A-RESCUE-lora_sensor
- PICKIT1: footprint Socket_Strips:Socket_Strip_Straight_1x06_Pitch2.54mm -> Pin_Headers:Pin_Header_Straight_1x06_Pitch2.54mm
- UART2_CONN1: footprint Socket_Strips:Socket_Strip_Straight_1x03_Pitch2.54mm -> Pin_Headers:Pin_Header_Straight_1x03_Pitch2.54mm
Connections:
- net labels added: AN2_Temp, AN3_Ambient
- net labels removed: AN3_Temp
- wire segments 112 -> 113
Other:
- moved on the sheet: C10, C11
Changed lines of the file:
@@
 LIBS:mcp9700t-e
 LIBS:rn2483
+LIBS:fa_238
 LIBS:lora_sensor-cache
-EELAYER 25 0
+EELAYER 26 0
 EELAYER END
 $Descr A4 11693 8268
@@
 F 0 "PICKIT1" H 3950 2000 50  0000 C CNN
 F 1 "CONN_01X06" V 4050 1650 50  0000 C CNN
-F 2 "Socket_Strips:Socket_Strip_Straight_1x06_Pitch2.54mm" H 3950 1650 50  0001 C CNN
+F 2 "Pin_Headers:Pin_Header_Straight_1x06_Pitch2.54mm" H 3950 1650 50  0001 C CNN
 F 3 "" H 3950 1650 50  0000 C CNN
 	1    3950 1650
@@
 VPP/~MCLR
 $Comp
-L USB_A P1
+L USB_A-RESCUE-lora_sensor P1
 U 1 1 589BC9B4
 P 2800 6450
@@
 Text Label 4300 4350 0    60   ~ 0
 OSC2
-Text Label 1050 3550 0    60   ~ 0
+Text Label 750  3550 0    60   ~ 0
 OSC1
-Text Label 1900 3550 0    60   ~ 0
+Text Label 2000 3550 0    60   ~ 0
 OSC2
-$Comp
-L Crystal_GND23 Y1
-U 1 1 589BCA0D
-P 1550 3550
-F 0 "Y1" H 1675 3750 50  0000 L CNN
-F 1 "16Mhz" H 1675 3675 50  0000 L CNN
-F 2 "Crystals:Crystal_SMD_EuroQuartz_MQ-4pin_7.0x5.0mm_HandSoldering" H 1550 3550 50  0001 C CNN
-F 3 "" H 1550 3550 50  0000 C CNN
-	1    1550 3550
-	1    0    0    -1
-$EndComp
 $Comp
 L GND #PWR027
 U 1 1 589BCA14
-P 1550 4100
-F 0 "#PWR027" H 1550 3850 50  0001 C CNN
-F 1 "GND" H 1550 3950 50  0000 C CNN
-F 2 "" H 1550 4100 50  0000 C CNN
-F 3 "" H 1550 4100 50  0000 C CNN
-	1    1550 4100
+P 1650 4100
+F 0 "#PWR027" H 1650 3850 50  0001 C CNN
+F 1 "GND" H 1650 3950 50  0000 C CNN
+F 2 "" H 1650 4100 50  0000 C CNN
+F 3 "" H 1650 4100 50  0000 C CNN
+	1    1650 4100
 	1    0    0    -1
 $EndComp
@@
 L C C11
 U 1 1 589BCA1A
-P 1800 3800
-F 0 "C11" H 1825 3900 50  0000 L CNN
-F 1 "22pF" H 1825 3700 50  0000 L CNN
-F 2 "Capacitors_SMD:C_0805" H 1838 3650 50  0001 C CNN
-F 3 "" H 1800 3800 50  0000 C CNN
-	1    1800 3800
+P 2350 3800
+F 0 "C11" H 2375 3900 50  0000 L CNN
+F 1 "22pF" H 2375 3700 50  0000 L CNN
+F 2 "Capacitors_SMD:C_0805" H 2388 3650 50  0001 C CNN
+F 3 "" H 2350 3800 50  0000 C CNN
+	1    2350 3800
 	1    0    0    -1
 $EndComp
@@
 L C C10
 U 1 1 589BCA21
-P 1300 3800
-F 0 "C10" H 1325 3900 50  0000 L CNN
-F 1 "22pF" H 1325 3700 50  0000 L CNN
-F 2 "Capacitors_SMD:C_0805" H 1338 3650 50  0001 C CNN
-F 3 "" H 1300 3800 50  0000 C CNN
-	1    1300 3800
+P 700 3800
+F 0 "C10" H 725 3900 50  0000 L CNN
+F 1 "22pF" H 725 3700 50  0000 L CNN
+F 2 "Capacitors_SMD:C_0805" H 738 3650 50  0001 C CNN
+F 3 "" H 700 3800 50  0000 C CNN
+	1    700  3800
 	1    0    0    -1
 $EndComp
 $Comp
 L GND #PWR028
-U 1 1 589BCA28
-P 1750 3150
-F 0 "#PWR028" H 1750 2900 50  0001 C CNN
-F 1 "GND" H 1750 3000 50  0000 C CNN
-F 2 "" H 1750 3150 50  0000 C CNN
-F 3 "" H 1750 3150 50  0000 C CNN
-	1    1750 3150
-	1    0    0    -1
-$EndComp
-$Comp
-L GND #PWR029
 U 1 1 589BCA2E
 P 4300 6600
-F 0 "#PWR029" H 4300 6350 50  0001 C CNN
+F 0 "#PWR028" H 4300 6350 50  0001 C CNN
 F 1 "GND" H 4300 6450 50  0000 C CNN
 F 2 "" H 4300 6600 50  0000 C CNN
@@
 F 0 "UART2_CONN1" H 7900 1700 50  0000 C CNN
 F 1 "CONN_01X03" V 8000 1500 50  0000 C CNN
-F 2 "Socket_Strips:Socket_Strip_Straight_1x03_Pitch2.54mm" H 7900 1500 50  0001 C CNN
+F 2 "Pin_Headers:Pin_Header_Straight_1x03_Pitch2.54mm" H 7900 1500 50  0001 C CNN
 F 3 "" H 7900 1500 50  0000 C CNN
 	1    7900 1500
@@
 $EndComp
 $Comp
-L GND #PWR030
+L GND #PWR029
 U 1 1 589BCA42
 P 7600 1700
-F 0 "#PWR030" H 7600 1450 50  0001 C CNN
+F 0 "#PWR029" H 7600 1450 50  0001 C CNN
 F 1 "GND" H 7600 1550 50  0000 C CNN
 F 2 "" H 7600 1700 50  0000 C CNN
@@
 UART_2_TX
 $Comp
-L LED LED3
+L LED-RESCUE-lora_sensor LED3
 U 1 1 589BCA4A
 P 10850 4500
+AR Path="/589BCA4A" Ref="LED3"  Part="1"
+AR Path="/5899E253/589BCA4A" Ref="LED3"  Part="1"
 F 0 "LED3" H 10850 4600 50  0000 C CNN
 F 1 "LED" H 10850 4400 50  0000 C CNN
@@
 $EndComp
 $Comp
-L LED LED2
+L LED-RESCUE-lora_sensor LED2
 U 1 1 589BCA51
 P 10550 4500
+AR Path="/589BCA51" Ref="LED2"  Part="1"
+AR Path="/5899E253/589BCA51" Ref="LED2"  Part="1"
 F 0 "LED2" H 10550 4600 50  0000 C CNN
 F 1 "LED" H 10550 4400 50  0000 C CNN
@@
 $EndComp
 $Comp
-L LED LED1
+L LED-RESCUE-lora_sensor LED1
 U 1 1 589BCA6D
 P 10250 4500
+AR Path="/589BCA6D" Ref="LED1"  Part="1"
+AR Path="/5899E253/589BCA6D" Ref="LED1"  Part="1"
 F 0 "LED1" H 10250 4600 50  0000 C CNN
 F 1 "LED" H 10250 4400 50  0000 C CNN
@@
 $EndComp
 $Comp
-L LED LED0
+L LED-RESCUE-lora_sensor LED0
 U 1 1 589BCA74
 P 9950 4500
+AR Path="/589BCA74" Ref="LED0"  Part="1"
+AR Path="/5899E253/589BCA74" Ref="LED0"  Part="1"
 F 0 "LED0" H 9950 4600 50  0000 C CNN
 F 1 "LED" H 9950 4400 50  0000 C CNN
@@
 $EndComp
 $Comp
-L GND #PWR031
+L GND #PWR030
 U 1 1 589BCA82
 P 10850 4750
-F 0 "#PWR031" H 10850 4500 50  0001 C CNN
+F 0 "#PWR030" H 10850 4500 50  0001 C CNN
 F 1 "GND" H 10850 4600 50  0000 C CNN
 F 2 "" H 10850 4750 50  0000 C CNN
@@
 V_CAP
 $Comp
-L GND #PWR032
+L GND #PWR031
 U 1 1 589BCA8B
 P 4850 1600
-F 0 "#PWR032" H 4850 1350 50  0001 C CNN
+F 0 "#PWR031" H 4850 1350 50  0001 C CNN
 F 1 "GND" H 4850 1450 50  0000 C CNN
 F 2 "" H 4850 1600 50  0000 C CNN
@@
 $EndComp
 $Comp
-L GND #PWR033
+L GND #PWR032
 U 1 1 589BCAA4
 P 10900 3000
-F 0 "#PWR033" H 10900 2750 50  0001 C CNN
+F 0 "#PWR032" H 10900 2750 50  0001 C CNN
 F 1 "GND" H 10900 2850 50  0000 C CNN
 F 2 "" H 10900 3000 50  0000 C CNN
@@
 $EndComp
 $Comp
-L GND #PWR034
+L GND #PWR033
 U 1 1 589BCABA
 P 10900 2250
-F 0 "#PWR034" H 10900 2000 50  0001 C CNN
+F 0 "#PWR033" H 10900 2000 50  0001 C CNN
 F 1 "GND" H 10900 2100 50  0000 C CNN
 F 2 "" H 10900 2250 50  0000 C CNN
@@
 Text Label 8050 3650 0    60   ~ 0
 Sensors_Enable
+Text Label 4300 3850 0    60   ~ 0
+AN3_Ambient
 Text Label 4300 3750 0    60   ~ 0
-AN2_Ambient
-Text Label 4300 3850 0    60   ~ 0
-AN3_Temp
+AN2_Temp
 Text Label 4300 4050 0    60   ~ 0
 RF_Reset
@@
 $EndComp
 $Comp
-L GND #PWR035
+L GND #PWR034
 U 1 1 589BCAD8
 P 4700 5150
-F 0 "#PWR035" H 4700 4900 50  0001 C CNN
+F 0 "#PWR034" H 4700 4900 50  0001 C CNN
 F 1 "GND" H 4700 5000 50  0000 C CNN
 F 2 "" H 4700 5150 50  0000 C CNN
@@
 	8550 3450 8000 3450
 Wire Wire Line
-	8000 3550 8550 3550
+	8000 3550 9300 3550
 Wire Wire Line
 	2750 3450 3550 3450
@@
 	4250 4350 4800 4350
 Wire Wire Line
-	1000 3550 1400 3550
-Wire Wire Line
-	1700 3550 2150 3550
-Wire Wire Line
-	1550 3750 1550 4100
-Wire Wire Line
-	1800 3650 1800 3550
-Connection ~ 1800 3550
-Wire Wire Line
-	1800 4050 1800 3950
-Wire Wire Line
-	1300 4050 1800 4050
-Connection ~ 1550 4050
-Wire Wire Line
-	1300 3950 1300 4050
-Wire Wire Line
-	1300 3650 1300 3550
-Connection ~ 1300 3550
-Wire Wire Line
-	1550 3350 1550 3050
-Wire Wire Line
-	1550 3050 1750 3050
-Wire Wire Line
-	1750 3050 1750 3150
+	700  3550 1200 3550
+Wire Wire Line
+	1800 3550 2350 3550
+Wire Wire Line
+	700  4050 2350 4050
 Wire Wire Line
 	7600 1700 7600 1600
@@
 	8000 3650 8750 3650
 Wire Wire Line
-	4250 3750 4800 3750
-Wire Wire Line
-	4800 3850 4250 3850
+	4250 3850 4800 3850
+Wire Wire Line
+	4800 3750 4250 3750
 Wire Wire Line
 	4250 4050 4800 4050
@@
 Text Label 1550 2100 0    60   ~ 0
 AN1_LDR
-Text Label 1550 2200 0    60   ~ 0
-AN2_Ambient
-Text Label 1550 2300 0    60   ~ 0
-AN3_Temp
 Wire Wire Line
 	1500 2000 2050 2000
 Wire Wire Line
 	2050 2100 1500 2100
-Wire Wire Line
-	1500 2200 2050 2200
-Wire Wire Line
-	2050 2300 1500 2300
 Text HLabel 1500 2000 0    60   Input ~ 0
 AN0_Battery
@@
 V_USB
 $Comp
-L GND #PWR036
+L GND #PWR035
 U 1 1 589BCB64
 P 1600 1250
-F 0 "#PWR036" H 1600 1000 50  0001 C CNN
+F 0 "#PWR035" H 1600 1000 50  0001 C CNN
 F 1 "GND" H 1600 1100 50  0000 C CNN
 F 2 "" H 1600 1250 50  0000 C CNN
@@
 Text Notes 9300 5150 0    60   ~ 0
 The LED resistor values can be adjusted \nbased on the LEDs that are used.
+Wire Wire Line
+	700  3650 700  3550
+Wire Wire Line
+	700  3950 700  4050
+Wire Wire Line
+	2350 4050 2350 3950
+Wire Wire Line
+	2350 3550 2350 3650
+Connection ~ 1800 4050
+Connection ~ 1150 4050
+Wire Wire Line
+	1650 4100 1650 4050
+Connection ~ 1650 4050
+Wire Wire Line
+	1800 3750 1900 3750
+Wire Wire Line
+	1900 3750 1900 4050
+Connection ~ 1900 4050
+Wire Wire Line
+	1200 3750 1150 3750
+Wire Wire Line
+	1150 3750 1150 4050
+Text Label 1550 2200 0    60   ~ 0
+AN3_Ambient
+Text Label 1550 2300 0    60   ~ 0
+AN2_Temp
+Wire Wire Line
+	1500 2200 2050 2200
+Wire Wire Line
+	2050 2300 1500 2300
+Text Label 8650 3550 0    60   ~ 0
+BUTTON_1
+$Comp
+L FA_238 Y1
+U 1 1 589F0EF6
+P 1500 3550
+F 0 "Y1" H 1500 3943 60  0000 C CNN
+F 1 "FA_238" H 1500 3837 60  0000 C CNN
+F 2 "libraries:Crystal_FA-238" H 1500 3731 60  0000 C CNN
+F 3 "" H -50 200 60  0000 C CNN
+	1    1500 3550
+	1    0    0    -1
+$EndComp
 $EndSCHEMATC
