File: pcb_layout/rf_section.sch (KiCad schematic (older format))
At the start: 14 parts, among them U1 RN2483

Commit message: More modules, initial pcb layout
Parts:
- R3, R4: value R -> 330
- RF_High1, RF_Low1: footprint (none) -> libraries:SMA_edge_connect
- renumbered RF_LED_1 to RF_LED_0, RF_LED_2 to RF_LED_1
Changed lines of the file:
@@
 F 0 "RF_High1" V 5350 2450 50  0000 C CNN
 F 1 "CONN_01X02" V 5250 2450 50  0000 C CNN
-F 2 "" H 5150 2450 50  0001 C CNN
+F 2 "libraries:SMA_edge_connect" H 5150 2450 50  0001 C CNN
 F 3 "" H 5150 2450 50  0000 C CNN
 	1    5150 2450
@@
 F 0 "RF_Low1" V 4950 2450 50  0000 C CNN
 F 1 "CONN_01X02" V 4850 2450 50  0000 C CNN
-F 2 "" H 4750 2450 50  0001 C CNN
+F 2 "libraries:SMA_edge_connect" H 4750 2450 50  0001 C CNN
 F 3 "" H 4750 2450 50  0000 C CNN
 	1    4750 2450
@@
 RF_POW
 $Comp
-L GND #PWR7
+L GND #PWR01
 U 1 1 589AAC19
 P 8600 2250
-F 0 "#PWR7" H 8600 2000 50  0001 C CNN
+F 0 "#PWR01" H 8600 2000 50  0001 C CNN
 F 1 "GND" H 8600 2100 50  0000 C CNN
 F 2 "" H 8600 2250 50  0000 C CNN
@@
 NoConn ~ 5850 4900
 $Comp
-L LED RF_LED_2
+L LED RF_LED_1
 U 1 1 589AAC25
 P 8300 5050
-F 0 "RF_LED_2" H 8300 5150 50  0000 C CNN
+F 0 "RF_LED_1" H 8300 5150 50  0000 C CNN
 F 1 "LED" H 8300 4950 50  0000 C CNN
 F 2 "LEDs:LED_0805" H 8300 5050 50  0001 C CNN
@@
 $EndComp
 $Comp
-L LED RF_LED_1
+L LED RF_LED_0
 U 1 1 589AAC2C
 P 8000 5050
-F 0 "RF_LED_1" H 8000 5150 50  0000 C CNN
+F 0 "RF_LED_0" H 8000 5150 50  0000 C CNN
 F 1 "LED" H 8000 4950 50  0000 C CNN
 F 2 "LEDs:LED_0805" H 8000 5050 50  0001 C CNN
@@
 P 8300 4650
 F 0 "R4" V 8380 4650 50  0000 C CNN
-F 1 "R" V 8300 4650 50  0000 C CNN
+F 1 "330" V 8300 4650 50  0000 C CNN
 F 2 "Resistors_SMD:R_0805" V 8230 4650 50  0001 C CNN
 F 3 "" H 8300 4650 50  0000 C CNN
@@
 P 8000 4650
 F 0 "R3" V 8080 4650 50  0000 C CNN
-F 1 "R" V 8000 4650 50  0000 C CNN
+F 1 "330" V 8000 4650 50  0000 C CNN
 F 2 "Resistors_SMD:R_0805" V 7930 4650 50  0001 C CNN
 F 3 "" H 8000 4650 50  0000 C CNN
@@
 $EndComp
 $Comp
-L GND #PWR5
+L GND #PWR02
 U 1 1 589AAC61
 P 7950 3550
-F 0 "#PWR5" H 7950 3300 50  0001 C CNN
+F 0 "#PWR02" H 7950 3300 50  0001 C CNN
 F 1 "GND" H 7950 3400 50  0000 C CNN
 F 2 "" H 7950 3550 50  0000 C CNN
@@
 $EndComp
 $Comp
-L GND #PWR8
+L GND #PWR03
 U 1 1 589AAC67
 P 8850 3550
-F 0 "#PWR8" H 8850 3300 50  0001 C CNN
+F 0 "#PWR03" H 8850 3300 50  0001 C CNN
 F 1 "GND" H 8850 3400 50  0000 C CNN
 F 2 "" H 8850 3550 50  0000 C CNN
@@
 	4050 3800 3550 3800
 $Comp
-L GND #PWR6
+L GND #PWR04
 U 1 1 589AACC1
 P 8150 5300
-F 0 "#PWR6" H 8150 5050 50  0001 C CNN
+F 0 "#PWR04" H 8150 5050 50  0001 C CNN
 F 1 "GND" H 8150 5150 50  0000 C CNN
 F 2 "" H 8150 5300 50  0000 C CNN
@@
 	1900 1650 2400 1650
 $Comp
-L GND #PWR1
+L GND #PWR05
 U 1 1 589AB2FF
 P 2000 1850
-F 0 "#PWR1" H 2000 1600 50  0001 C CNN
+F 0 "#PWR05" H 2000 1600 50  0001 C CNN
 F 1 "GND" H 2000 1700 50  0000 C CNN
 F 2 "" H 2000 1850 50  0000 C CNN
@@
 Connection ~ 3250 5300
 $Comp
-L GND #PWR2
+L GND #PWR06
 U 1 1 58978DB5
 P 3250 5450
-F 0 "#PWR2" H 3250 5200 50  0001 C CNN
+F 0 "#PWR06" H 3250 5200 50  0001 C CNN
 F 1 "GND" H 3250 5300 50  0000 C CNN
 F 2 "" H 3250 5450 50  0000 C CNN
@@
 $EndComp
 $Comp
-L GND #PWR4
+L GND #PWR07
 U 1 1 58978FDA
 P 6500 5450
-F 0 "#PWR4" H 6500 5200 50  0001 C CNN
+F 0 "#PWR07" H 6500 5200 50  0001 C CNN
 F 1 "GND" H 6500 5300 50  0000 C CNN
 F 2 "" H 6500 5450 50  0000 C CNN
@@
 Connection ~ 6500 4300
 $Comp
-L GND #PWR3
+L GND #PWR08
 U 1 1 5897BB26
 P 5950 2900
-F 0 "#PWR3" H 5950 2650 50  0001 C CNN
+F 0 "#PWR08" H 5950 2650 50  0001 C CNN
 F 1 "GND" H 5950 2750 50  0000 C CNN
 F 2 "" H 5950 2900 50  0000 C CNN

Commit message: Added PCB LAyout
Parts:
- RF_LED_0, RF_LED_1: symbol LED -> LED-RESCUE-lora_sensor
- renumbered RF_High1 to RF_HIGH_1, RF_Low1 to RF_LOW_1
Changed lines of the file:
@@
 LIBS:mcp9700t-e
 LIBS:rn2483
+LIBS:fa_238
 LIBS:lora_sensor-cache
-EELAYER 25 0
+EELAYER 26 0
 EELAYER END
 $Descr A4 11693 8268
@@
 NoConn ~ 4050 3500
 $Comp
-L CONN_01X02 RF_High1
+L CONN_01X02 RF_HIGH_1
 U 1 1 589AABF6
 P 5150 2450
-F 0 "RF_High1" V 5350 2450 50  0000 C CNN
+F 0 "RF_HIGH_1" V 5350 2450 50  0000 C CNN
 F 1 "CONN_01X02" V 5250 2450 50  0000 C CNN
 F 2 "libraries:SMA_edge_connect" H 5150 2450 50  0001 C CNN
@@
 $EndComp
 $Comp
-L CONN_01X02 RF_Low1
+L CONN_01X02 RF_LOW_1
 U 1 1 589AABFD
 P 4750 2450
-F 0 "RF_Low1" V 4950 2450 50  0000 C CNN
+F 0 "RF_LOW_1" V 4950 2450 50  0000 C CNN
 F 1 "CONN_01X02" V 4850 2450 50  0000 C CNN
 F 2 "libraries:SMA_edge_connect" H 4750 2450 50  0001 C CNN
@@
 NoConn ~ 5850 4900
 $Comp
-L LED RF_LED_1
+L LED-RESCUE-lora_sensor RF_LED_1
 U 1 1 589AAC25
 P 8300 5050
+AR Path="/589AAC25" Ref="RF_LED_1"  Part="1"
+AR Path="/58974944/589AAC25" Ref="RF_LED_1"  Part="1"
 F 0 "RF_LED_1" H 8300 5150 50  0000 C CNN
 F 1 "LED" H 8300 4950 50  0000 C CNN
@@
 $EndComp
 $Comp
-L LED RF_LED_0
+L LED-RESCUE-lora_sensor RF_LED_0
 U 1 1 589AAC2C
 P 8000 5050
+AR Path="/589AAC2C" Ref="RF_LED_0"  Part="1"
+AR Path="/58974944/589AAC2C" Ref="RF_LED_0"  Part="1"
 F 0 "RF_LED_0" H 8000 5150 50  0000 C CNN
 F 1 "LED" H 8000 4950 50  0000 C CNN
