File: pcb_layout/sensor_section.sch (KiCad schematic (older format))
At the start: 10 parts, among them Q2 NXP 2N7002,215, Q3 NXP BSS84, U5 BH1603FVC, U6 MCP9700T-E

Commit message: More modules, initial pcb layout
Parts:
- U5: footprint (none) -> libraries:BH1603FVC
Changed lines of the file:
@@
 $EndComp
 $Comp
-L GND #PWR38
+L GND #PWR037
 U 1 1 589BF0F5
 P 2350 4400
-F 0 "#PWR38" H 2350 4150 50  0001 C CNN
+F 0 "#PWR037" H 2350 4150 50  0001 C CNN
 F 1 "GND" H 2350 4250 50  0000 C CNN
 F 2 "" H 2350 4400 50  0000 C CNN
@@
 $EndComp
 $Comp
-L GND #PWR41
+L GND #PWR038
 U 1 1 589BF10C
 P 7400 4300
-F 0 "#PWR41" H 7400 4050 50  0001 C CNN
+F 0 "#PWR038" H 7400 4050 50  0001 C CNN
 F 1 "GND" H 7400 4150 50  0000 C CNN
 F 2 "" H 7400 4300 50  0000 C CNN
@@
 F 0 "U5" H 5900 3600 60  0000 C CNN
 F 1 "BH1603FVC" H 5900 4100 60  0000 C CNN
-F 2 "" H 5900 3850 60  0001 C CNN
+F 2 "libraries:BH1603FVC" H 5900 3850 60  0001 C CNN
 F 3 "" H 5900 3850 60  0001 C CNN
 	1    5900 3850
@@
 $EndComp
 $Comp
-L GND #PWR40
+L GND #PWR039
 U 1 1 589BF123
 P 5400 4000
-F 0 "#PWR40" H 5400 3750 50  0001 C CNN
+F 0 "#PWR039" H 5400 3750 50  0001 C CNN
 F 1 "GND" H 5400 3850 50  0000 C CNN
 F 2 "" H 5400 4000 50  0000 C CNN
@@
 $EndComp
 $Comp
-L GND #PWR39
+L GND #PWR040
 U 1 1 589BF139
 P 4750 4350
-F 0 "#PWR39" H 4750 4100 50  0001 C CNN
+F 0 "#PWR040" H 4750 4100 50  0001 C CNN
 F 1 "GND" H 4750 4200 50  0000 C CNN
 F 2 "" H 4750 4350 50  0000 C CNN
@@
 NoConn ~ 8750 3800
 $Comp
-L GND #PWR42
+L GND #PWR041
 U 1 1 589BF141
 P 8650 4100
-F 0 "#PWR42" H 8650 3850 50  0001 C CNN
+F 0 "#PWR041" H 8650 3850 50  0001 C CNN
 F 1 "GND" H 8650 3950 50  0000 C CNN
 F 2 "" H 8650 4100 50  0000 C CNN
@@
 	1950 1800 2650 1800
 $Comp
-L GND #PWR37
+L GND #PWR042
 U 1 1 589C714C
 P 2050 1450
-F 0 "#PWR37" H 2050 1200 50  0001 C CNN
+F 0 "#PWR042" H 2050 1200 50  0001 C CNN
 F 1 "GND" H 2050 1300 50  0000 C CNN
 F 2 "" H 2050 1450 50  0000 C CNN
